Commit message: Move laser scan to front lower

File: urdf/car_2d.urdf (robot description, URDF)
Before this commit: robot cartographer_backpack_2d, 3 links, 2 joints
Joints:
- joint horizontal_laser_link_joint: origin xyz=0.075 0 0.15 rpy=0 0 0 -> xyz=0.17 0 0.0 rpy=0 0 0

Commit message: Add rs200 frame

File: urdf/car_2d.urdf (robot description, URDF)
Before this commit: robot cartographer_backpack_2d, 3 links, 2 joints
Links:
- added link rs200; visual box size=0.01 0.13 0.02
Joints:
- added joint rs200_link_joint: type fixed, parent base_link, child rs200_frame, origin xyz=0.04 0 0.16 rpy=0 0 0

Commit message: fix typo

File: urdf/car_2d.urdf (robot description, URDF)
Before this commit: robot cartographer_backpack_2d, 4 links, 3 joints
Links:
- removed link rs200
- added link rs200_frame; visual box size=0.01 0.13 0.02

Commit message: FIx camera frame

File: urdf/car_2d.urdf (robot description, URDF)
Before this commit: robot cartographer_backpack_2d, 4 links, 3 joints
Joints:
- joint rs200_link_joint: origin xyz=0.04 0 0.16 rpy=0 0 0 -> xyz=0.04 0 0.16 rpy=3.14159 0 0

Commit message: Still fix camera frame

File: urdf/car_2d.urdf (robot description, URDF)
Before this commit: robot cartographer_backpack_2d, 4 links, 3 joints
Joints:
- joint rs200_link_joint: origin xyz=0.04 0 0.16 rpy=3.14159 0 0 -> xyz=0.04 0 0.16 rpy=0 -1.57079 0

Commit message: Correct with real data

File: urdf/car_2d.urdf (robot description, URDF)
Before this commit: robot cartographer_backpack_2d, 4 links, 3 joints
Joints:
- joint rs200_link_joint: origin xyz=0.04 0 0.16 rpy=0 -1.57079 0 -> xyz=0.04 0 0.195 rpy=-1.57079 0 1.57079

Commit message: Merge laser and camera frame for future use

File: urdf/car_2d.urdf (robot description, URDF)
Before this commit: robot cartographer_backpack_2d, 4 links, 3 joints
Links:
- added link camera_depth_optical_frame; visual box size=0.01 0.13 0.02
Joints:
- added joint laserr200_joint: type fixed, parent base_link, child camera_depth_optical_frame, origin xyz=0.04 0 0.195 rpy=0 0 3.141

Commit message: Fixed origin costmap raytrace problem by increasez

File: urdf/car_2d.urdf (robot description, URDF)
Before this commit: robot cartographer_backpack_2d, 5 links, 4 joints
Joints:
- joint horizontal_laser_link_joint: origin xyz=0.17 0 0.0 rpy=0 0 0 -> xyz=0.17 0 0.15 rpy=0 0 0
